Commit message: exer1_edit

File: students_copy/arm_urdf_pkg/urdf/panda.urdf (robot description, URDF)
Before this commit: robot panda, 12 links, 11 joints
Joints:
- joint panda_finger_joint1: type identify_joint_type -> IDENTIFY_JOINT_TYPE
- joint panda_finger_joint2: type identify_joint_type -> IDENTIFY_JOINT_TYPE
- joint panda_joint1: type revolute -> IDENTIFY_JOINT_TYPE
- joint panda_joint2: child panda_link2 -> IDENTIFY_CHILD_LINK; parent panda_link1 -> IDENTIFY_PARENT_LINK; type revolute -> IDENTIFY_JOINT_TYPE
- joint panda_joint3: child panda_link3 -> IDENTIFY_CHILD_LINK; parent panda_link2 -> IDENTIFY_PARENT_LINK; type revolute -> IDENTIFY_JOINT_TYPE
- joint panda_joint4: child panda_link4 -> IDENTIFY_CHILD_LINK; parent panda_link3 -> IDENTIFY_PARENT_LINK; type revolute -> IDENTIFY_JOINT_TYPE
- joint panda_joint5: child panda_link5 -> IDENTIFY_CHILD_LINK; parent panda_link4 -> IDENTIFY_PARENT_LINK; type revolute -> IDENTIFY_JOINT_TYPE
- joint panda_joint6: type revolute -> IDENTIFY_JOINT_TYPE
- joint panda_joint7: type revolute -> IDENTIFY_JOINT_TYPE
